File: HARDWARE/FOSDEM-MUSIC-BOX_RevA/FOSDEM-MUSIC-BOX_RevA.sch (KiCad schematic (older format))
At the start: 23 parts, among them SW1 T1101GP(6x3x4.3MM), U1 ATTINY85-20PU, U2 LM386N

Commit message: Update
Parts:
- R7: value 1.5K -> 10K
- R9: value 10K -> 1.5K

Commit message: Update
Parts:
- R10: value 1.5K -> 10K
Changed lines of the file:
@@
 P 3600 2000
 F 0 "R10" V 3500 2100 50  0000 L CNN
-F 1 "1.5K" V 3700 2100 50  0000 L CNN
+F 1 "10K" V 3700 2100 50  0000 L CNN
 F 2 "Resistor_THT:R_Axial_DIN0204_L3.6mm_D1.6mm_P7.62mm_Horizontal" H 3600 1930 30  0001 C CNN
 F 3 "" V 3600 2000 30  0000 C CNN
